File: _autosave-USBpowermeter.kicad_pcb (KiCad board)
At the start: 2 copper layers, 65 parts, among them J1 USB4215-03-A, J3 FPC-05FB-30PH20, J4 HX PZ1.27-2X7P TP, J5 USB4155-03-C, Q1 2N7002K_C414015, Q2 BRCS5P06MA, Q3 FDN338P_C347511, Q4 FDN335N, SW3 TS24CA, SW4 TS24CA, SW5 MINI MSK12CO2, SW6 TS24CA, U1 STM32G030K6T6TR, U2 INA238AIDGSR, U3 LMR36006FSC3RNXRQ1, U7 TLV61046ADBVR

Commit message: schematic changes
Parts:
- added C11: 100nF, Capacitor_SMD:C_0402_1005Metric, F.Cu at (106.9, 84.6)
- added L2: 10uH, Inductor_SMD:L_0603_1608Metric, F.Cu at (110.6, 78.8)
- added R26: 10kΩ, Resistor_SMD:R_0402_1005Metric, F.Cu at (110.6, 111.0)
- added R4: 10R, Resistor_SMD:R_0402_1005Metric, F.Cu at (110.0, 81.0)
- added R5: 10R, Resistor_SMD:R_0402_1005Metric, F.Cu at (110.0, 83.0)
- added TP18: TP4, TestPoint:TestPoint_Pad_D1.0mm, F.Cu at (105.0, 111.0)
- added TP20: TP4, TestPoint:TestPoint_Pad_D1.0mm, F.Cu at (108.1, 111.0)
- added TP21: TP4, TestPoint:TestPoint_Pad_D1.0mm, F.Cu at (105.0, 107.9)
- added TP22: TP4, TestPoint:TestPoint_Pad_D1.0mm, F.Cu at (108.1, 107.9)
- added TP23: TP4, TestPoint:TestPoint_Pad_D1.0mm, F.Cu at (105.0, 104.9)
- added TP24: TP4, TestPoint:TestPoint_Pad_D1.0mm, F.Cu at (108.1, 104.9)
- added TP25: TP4, TestPoint:TestPoint_Pad_D1.0mm, F.Cu at (105.0, 101.8)
- added TP26: TP4, TestPoint:TestPoint_Pad_D1.0mm, F.Cu at (108.1, 101.8)
- added TP27: TP4, TestPoint:TestPoint_Pad_D1.0mm, F.Cu at (107.0, 79.0)
- added TP28: TP4, TestPoint:TestPoint_Pad_D1.0mm, F.Cu at (107.0, 82.1)
Connections:
- J4 pad 1: +3.3V -> unconnected-(J4-Pad1)
- J4 pad 10: /NRST -> unconnected-(J4-Pad10)
- J4 pad 11: unconnected-(J4-Pad11) -> GND
- J4 pad 12: unconnected-(J4-Pad12) -> /NRST
- J4 pad 2: /SWDIO -> unconnected-(J4-Pad2)
- J4 pad 3: GND -> +3.3V
- J4 pad 4: /SWCLK -> /SWDIO
- J4 pad 6: unconnected-(J4-Pad6) -> /SWCLK
- J4 pad 7: unconnected-(J4-Pad7) -> GND
- J4 pad 9: GND -> unconnected-(J4-Pad9)
- U1 pad 12: /BUZZER_DRIVE -> unconnected-(U1-PA5-Pad12)
- U1 pad 15: unconnected-(U1-PB0-Pad15) -> /BUZZER_DRIVE
- U2 pad 10: VBUS_SW -> Net-(U2-IN+)
- U2 pad 8: VBUS_OUT -> Net-(U2-IN-)
- U2 pad 9: VBUS_OUT -> Net-(U2-IN-)
- U3 pad 9: /BUCK_EN -> VBUS_SW
