File: USBpowermeter.kicad_sch (KiCad schematic)
At the start: 73 parts, among them J1 USB4215-03-A, J2 2188470001, J3 FPC-05FB-30PH20, J4 HX PZ1.27-2X7P TP, Q1 2N7002K_C414015, Q2 BRCS5P06MA, Q3 FDN338P_C347511, Q4 FDN335N, SW1 TS24CA, SW2 TS24CA, SW4 TS24CA, SW5 MINI MSK12CO2, U1 STM32G030K6T6TR, U2 INA238AIDGSR, U3 LMR36006FSC3RNXRQ1, U7 TLV61046ADBVR

Commit message: Schem update
Parts:
- removed C16, C17, C23: 10nF, symbol Device:C_Small
- removed J1: USB4215-03-A, Library:USB-C-SMD_GT-USB-7010B, symbol Library:USB4215-03-A
- removed J2: 2188470001, Library:USB-C-SMD_TYPEC-952-ACP24, symbol Library:2188470001
- removed R10, R11, R22: 10kΩ, symbol Device:R_Small
- removed SW1, SW2: TS24CA, Library:SW-SMD_2P-TS24CA, symbol Library:TS24CA
- removed TP20: TP6, symbol Connector:TestPoint
- removed TP21: TP7, symbol Connector:TestPoint
- added C24, C29, C30: 10nF, symbol Device:C_Small
- added J1: USB4215-03-A, Library_new:CONN_8p94X6p5X3p16_12L_GCC, symbol USB4215:USB4215-03-A
- added J5: USB4155-03-C_REVA, Library_new:GCT_USB4155-03-C_REVA, symbol USB4155-03-C_REVA:USB4155-03-C_REVA
- added R23, R24, R25: 10kΩ, symbol Device:R_Small
- added SW3, SW6: TS24CA, Library:SW-SMD_2P-TS24CA, symbol Library:TS24CA
Connections:
- net +3.3V: now also R23.1, R24.1, R25.1
- net BTN_AUX: now also C30.2, R25.2, SW6.2; no longer SW4.1, SW4.3
- net BTN_PAGE: now also C24.2, R23.2, SW3.2
- net BTN_RESET: now also SW4.2, C29.2, R24.2
- net CC1_PASS: now also J1.A5 (CC1), J5.A5 (CC1)
- net CC2_PASS: now also J1.B5 (CC2), J5.B5 (CC2)
- net GND: now also SW4.1, C24.1, C29.1, C30.1, J1.13 (GND), J1.14 (GND), J1.15 (GND), J1.16 (GND), J1.A1/B12 (GND), J1.B1/A12 (GND), J5.A1 (GND_A), J5.A12 (GND_A__1), J5.B1 (GND_B), J5.B12 (GND_B__1), J5.S1 (SHELL_GND), J5.S2 (SHELL_GND__1), SW3.1, SW6.1; no longer SW4.2, SW4.4
- net SBU1_PASS: now also J1.A8 (SBU1), J5.A8 (SBU1)
- net SBU2_PASS: now also J1.B8 (SBU2), J5.B8 (SBU2)
- net USB2_DN: now also J1.A7 (DN1), J1.B7 (DN2), J5.A7 (DN1), J5.B7 (DN2)
- net USB2_DP: now also J1.A6 (DP1), J1.B6 (DP2), J5.A6 (DP1), J5.B6 (DP2)
- net VBUS_IN: now also J1.A4/B9 (VBUS), J1.B4/A9 (VBUS)
- net VBUS_OUT: now also J5.A4 (VBUS_A), J5.A9 (VBUS_A__1), J5.B4 (VBUS_B), J5.B9 (VBUS_B__1)
Other:
- added sheet STM32 (STM32.kicad_sch.kicad_sch)
- added sheet STM33 (STM32.kicad_sch.kicad_sch)
- added sheet USB-C FEMALE (USB_C_FEMALE.kicad_sch.kicad_sch)
- added sheet USB-C MALE (USB_C_MALE.kicad_sch.kicad_sch)
- moved on the sheet: BZ1, C1, C10, C12, C13, C14, C15, C18, C19, C2, C20, C21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

Commit message: schematic changes
Parts:
- removed C14: 100nF, Capacitor_SMD:C_0805_2012Metric, symbol Device:C_Small
- removed C18: 100nF, symbol Device:C_Small
- removed C19: 1uF, symbol Device:C_Small
- removed C20: 4.7uF, symbol Device:C_Small
- removed D3: SMAJ58CA_C2943847, Library:SMA_L4.2-W2.6-LS5.0-BI, symbol Library:SMAJ58CA_C2943847
- removed R17: 38.3kΩ, symbol Device:R_Small
- removed R18: 10kΩ, symbol Device:R_Small
- removed R6: 1MΩ, symbol Device:R_Small
- removed TP1: TP1, TestPoint:TestPoint_Pad_D1.5mm, symbol Connector:TestPoint
- removed TP12: TP12, TestPoint:TestPoint_Pad_D1.5mm, symbol Connector:TestPoint
- removed TP2: TP2, TestPoint:TestPoint_Pad_D1.5mm, symbol Connector:TestPoint
- removed U7: TLV61046ADBVR, Library:SOT-23-6_L2.9-W1.6-P0.95-LS2.8-BL, symbol Library:TLV61046ADBVR
- added C11, C23: 100nF, Capacitor_SMD:C_0402_1005Metric, symbol Device:C_Small
- added C16, C17: 10uF, Capacitor_SMD:C_0402_1005Metric, symbol Device:C_Small
- added R10: 215k, Resistor_SMD:R_0402_1005Metric, symbol Device:R_Small
- added R26: 10kΩ, Resistor_SMD:R_0402_1005Metric, symbol Device:R_Small
- added R4: 10R, Resistor_SMD:R_0402_1005Metric, symbol Device:R_Small
- added R8: 100kΩ, Resistor_SMD:R_0402_1005Metric, symbol Device:R_Small
- added TP18, TP20, TP21, TP22, TP23, TP24, TP25, TP27, TP28: TP4, TestPoint:TestPoint_Pad_D1.0mm, symbol Connector:TestPoint
- added U4: MSMCP1640T-I/CHY, Package_TO_SOT_SMD:SOT-23-6, symbol New_Library:MSMCP1640T-I/CHY
- BZ1: value FST-9650B-3V -> MLT-5020; footprint Library:BUZ-SMD_L9.6-W9.6-LS10.0-R -> C94598:BUZ-SMD_L5.0-W5.5-P4.60; LCSC Part (none) -> C94598
- C1: footprint (none) -> Capacitor_SMD:C_0603_1608Metric; LCSC Part (none) -> C77058
- C10, C12, C13, C2, C27, C28, C4, C6: footprint (none) -> Capacitor_SMD:C_0402_1005Metric; LCSC Part (none) -> C42371686
- C15, C21: footprint (none) -> Capacitor_SMD:C_0402_1005Metric; LCSC Part (none) -> C15525
- C22, C3, C5, C9: footprint (none) -> Capacitor_SMD:C_0402_1005Metric; LCSC Part (none) -> C343042
- C24, C29, C30: footprint (none) -> Capacitor_SMD:C_0402_1005Metric; LCSC Part (none) -> C22400107
- C25: footprint (none) -> Capacitor_SMD:C_0402_1005Metric; LCSC Part (none) -> C318563
- C26: footprint (none) -> Capacitor_SMD:C_0402_1005Metric; LCSC Part (none) -> C12530
- D1: LCSC Part (none) -> C148235
- D4: LCSC Part (none) -> C19077410
- J1: LCSC Part (none) -> C37616412
- J3: Display (none) -> X096-2864KSWPG01-H30; LCSC Part (none) -> C2856833
- J5: value USB4155-03-C_REVA -> USB4155-03-C; LCSC Part (none) -> ORDER ON DIGIKEY
- L1: footprint (none) -> Inductor_SMD:L_APV_ANR3015; LCSC Part (none) -> C6364792
- L2: value 10uH -> 4.7uH; footprint (none) -> Inductor_SMD:L_0603_1608Metric
- Q1: LCSC Part (none) -> C8545
- Q2: LCSC Part (none) -> C914070
- Q3: LCSC Part (none) -> C24855
- Q4: LCSC Part (none) -> C241804
- R1: footprint (none) -> Resistor_SMD:R_1206_3216Metric; LCSC Part (none) -> C2988648
- R12: footprint (none) -> Resistor_SMD:R_0402_1005Metric; LCSC Part (none) -> C2906860
- R13, R7: footprint (none) -> Resistor_SMD:R_0402_1005Metric; LCSC Part (none) -> C2906859
- R14, R23, R24, R25, R9: footprint (none) -> Resistor_SMD:R_0402_1005Metric; LCSC Part (none) -> C2906861
- R15: footprint (none) -> Resistor_SMD:R_0402_1005Metric; LCSC Part (none) -> C2909328
- R16: footprint (none) -> Resistor_SMD:R_0402_1005Metric; LCSC Part (none) -> C2909373
- R19: footprint (none) -> Resistor_SMD:R_0402_1005Metric; LCSC Part (none) -> C2909349
- R2, R3: footprint (none) -> Resistor_SMD:R_0402_1005Metric; LCSC Part (none) -> C105871
- R20, R21: footprint (none) -> Resistor_SMD:R_0402_1005Metric; LCSC Part (none) -> C2906872
- R5: value 100kΩ -> 10R; footprint (none) -> Resistor_SMD:R_0402_1005Metric; LCSC Part (none) -> C2906862
- SW3, SW4, SW6: LCSC Part (none) -> C393942
- SW5: LCSC Part (none) -> C2681570
- TP17, TP19: footprint (none) -> TestPoint:TestPoint_Pad_D1.0mm
- U1: footprint LIBRARY:LQFP-32_L7.0-W7.0-P0.80-LS9.0-BL -> Library:LQFP-32_L7.0-W7.0-P0.80-LS9.0-BL; LCSC Part (none) -> C724043
- U2: LCSC Part (none) -> C2868250
- U3: LCSC Part (none) -> C1850337
Connections:
- net +3.3V: now also J4.3, C16.1, C23.1, TP22.1, U4.6 (VIN); no longer J4.1
- net BUZZER_DRIVE: now also U1.15 (PB0); no longer U1.12 (PA5)
- net GND: now also J4.11, J4.7, SW3.3, SW3.4, SW4.3, SW4.4, SW6.3, SW6.4, C16.2, C17.2, C23.2, R26.2, R8.2, U4.2 (GND); no longer J4.3, J4.9
- net I2C_SCL: now also TP27.1
- net I2C_SDA: now also TP28.1
- net NRST: now also C22.1, J4.12, R14.2, U1.6 (NRST); no longer J4.10
- net OLED_3V8: now also C17.1, R10.1, TP23.1, U4.5 (VOUT)
- net OLED_POWER_EN: now also U4.3 (EN)
- net SWCLK: now also J4.6, U1.25 (PA14-BOOT0), R26.1; no longer J4.4
- net SWDIO: now also J4.4, U1.24 (PA13); no longer J4.2
- net VBUS_IN: now also D4.1 (K), Q2.2 (S), TP18.1; no longer Q2.3 (D)
- net VBUS_OUT: now also R5.2, TP25.1; no longer U2.8 (VBUS), U2.9 (IN-)
- net VBUS_SW: now also Q2.3 (D), U3.9 (EN), R4.2, TP20.1; no longer Q2.2 (S), R5.1, U2.10 (IN+)
- net at L2.2: now also U4.1 (LX)
- net at J3.6 (VDDB), Q3.3 (D): now also TP24.1
- net at D4.2 (A), Q2.1 (G), R15.2: now also SW5.2, TP21.1
- removed net BUCK_EN: R5.2, U3.9 (EN)
- new net: C11.2, R5.1, U2.8 (VBUS), U2.9 (IN-)
- new net: R10.2, R8.1, U4.4 (FB)
- new net: C11.1, R4.1, U2.10 (IN+)
Other:
- removed sheet STM32
- removed sheet STM33
- removed sheet USB-C FEMALE
- removed sheet USB-C MALE
- note added: "128x64 SSD1315 DISPLAY"
- note added: "BUZZER"
- note added: "HIGH-PRECISION POWER MONITOR"
- note added: "MAXIMUM RATINGS 46V, 5A Features: - OLED Screen - STM32G030 - INA238 Power Monitor"
- note added: "MENU CONFIG BUTTONS"
- note added: "OLED BOOST SUPPLY (3.8V)"
- note added: "POWER SWITCH"
- note added: "Rev 1"
- note added: "STM32 MCU"
- note added: "SWD Header"
- note added: "USB-C INPUT/OUTPUT CONNECTORS"
- note added: "USB-C Power Reader"
- note added: "VBUS->3V3 BUCK"
- note removed: "￼"
- moved on the sheet: BZ1, C1, C10, C12, C13, C15, C2, C21, C22, C24, C25, C26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

Commit message: push layout
Parts:
- added C18: 10uF, Capacitor_SMD:C_0805_2012Metric, symbol Device:C_Small
- L2: LCSC Part (none) -> C295681
- Q1, Q3, Q4: footprint Library:SOT-23-3_L2.9-W1.3-P1.90-LS2.4-BR -> Package_TO_SOT_SMD:SOT-23-3
- R10: LCSC Part (none) -> C3013158
Connections:
- net BTN_AUX: now also U1.12 (PA5); no longer U1.14 (PA7)
- net BTN_PAGE: now also U1.14 (PA7); no longer U1.7 (PA0)
- net BUCK_PG: now also U1.1 (PB9); no longer U1.11 (PA4)
- net GND: now also C18.2
- net OLED_RESET: now also U1.21 (PA10); no longer U1.9 (PA2)
- net VBUS_OUT: now also U2.8 (VBUS)
- net VBUS_SW: now also C18.1
- net at C11.2, R5.1, U2.9 (IN-): no longer U2.8 (VBUS)
- net USB2_DN renamed USB2_D-
- net USB2_DP renamed USB2_D+
