File: USBpowermeter.kicad_pcb (KiCad board)
At the start: 2 copper layers, 65 parts, among them J1 USB4215-03-A, J3 FPC-05FB-30PH20, J4 HX PZ1.27-2X7P TP, J5 USB4155-03-C, Q1 2N7002K_C414015, Q2 BRCS5P06MA, Q3 FDN338P_C347511, Q4 FDN335N, SW3 TS24CA, SW4 TS24CA, SW5 MINI MSK12CO2, SW6 TS24CA, U1 STM32G030K6T6TR, U2 INA238AIDGSR, U3 LMR36006FSC3RNXRQ1, U7 TLV61046ADBVR

Commit message: Changes
Parts:
- added C11: 100nF, Capacitor_SMD:C_0402_1005Metric, F.Cu at (106.9, 84.6)
- added L2: 10uH, Inductor_SMD:L_0603_1608Metric, F.Cu at (110.6, 78.8)
- added R26: 10kΩ, Resistor_SMD:R_0402_1005Metric, F.Cu at (110.6, 111.0)
- added R4: 10R, Resistor_SMD:R_0402_1005Metric, F.Cu at (110.0, 81.0)
- added R5: 10R, Resistor_SMD:R_0402_1005Metric, F.Cu at (110.0, 83.0)
- added TP18: TP4, TestPoint:TestPoint_Pad_D1.0mm, F.Cu at (105.0, 111.0)
- added TP20: TP4, TestPoint:TestPoint_Pad_D1.0mm, F.Cu at (108.1, 111.0)
- added TP21: TP4, TestPoint:TestPoint_Pad_D1.0mm, F.Cu at (105.0, 107.9)
- added TP22: TP4, TestPoint:TestPoint_Pad_D1.0mm, F.Cu at (108.1, 107.9)
- added TP23: TP4, TestPoint:TestPoint_Pad_D1.0mm, F.Cu at (105.0, 104.9)
- added TP24: TP4, TestPoint:TestPoint_Pad_D1.0mm, F.Cu at (108.1, 104.9)
- added TP25: TP4, TestPoint:TestPoint_Pad_D1.0mm, F.Cu at (105.0, 101.8)
- added TP26: TP4, TestPoint:TestPoint_Pad_D1.0mm, F.Cu at (108.1, 101.8)
- added TP27: TP4, TestPoint:TestPoint_Pad_D1.0mm, F.Cu at (107.0, 79.0)
- added TP28: TP4, TestPoint:TestPoint_Pad_D1.0mm, F.Cu at (107.0, 82.1)
Connections:
- J4 pad 1: +3.3V -> unconnected-(J4-Pad1)
- J4 pad 10: /NRST -> unconnected-(J4-Pad10)
- J4 pad 11: unconnected-(J4-Pad11) -> GND
- J4 pad 12: unconnected-(J4-Pad12) -> /NRST
- J4 pad 2: /SWDIO -> unconnected-(J4-Pad2)
- J4 pad 3: GND -> +3.3V
- J4 pad 4: /SWCLK -> /SWDIO
- J4 pad 6: unconnected-(J4-Pad6) -> /SWCLK
- J4 pad 7: unconnected-(J4-Pad7) -> GND
- J4 pad 9: GND -> unconnected-(J4-Pad9)
- U1 pad 12: /BUZZER_DRIVE -> unconnected-(U1-PA5-Pad12)
- U1 pad 15: unconnected-(U1-PB0-Pad15) -> /BUZZER_DRIVE
- U2 pad 10: VBUS_SW -> Net-(U2-IN+)
- U2 pad 8: VBUS_OUT -> Net-(U2-IN-)
- U2 pad 9: VBUS_OUT -> Net-(U2-IN-)
- U3 pad 9: /BUCK_EN -> VBUS_SW

Commit message: push layout
Parts:
- removed C19: 1uF, Capacitor_SMD:C_0402_1005Metric
- removed C20: 4.7uF, Capacitor_SMD:C_0402_1005Metric
- removed R17: 38.3kΩ, Resistor_SMD:R_0402_1005Metric
- removed R18: 10kΩ, Resistor_SMD:R_0402_1005Metric
- removed the R5 at (125.2, 93.1)
- removed R6: 1MΩ, Resistor_SMD:R_0402_1005Metric
- removed TP26: TP4, TestPoint:TestPoint_Pad_D1.0mm
- removed U7: TLV61046ADBVR, Library:SOT-23-6_L2.9-W1.6-P0.95-LS2.8-BL
- added C16: 10uF, Capacitor_SMD:C_0402_1005Metric, B.Cu at (70.0, 81.5)
- added C17: 10uF, Capacitor_SMD:C_0402_1005Metric, B.Cu at (72.5, 82.2)
- added C18: 10uF, Capacitor_SMD:C_0805_2012Metric, B.Cu at (90.1, 80.3)
- added R10: 215k, Resistor_SMD:R_0402_1005Metric, B.Cu at (74.3, 81.8)
- added R8: 100kΩ, Resistor_SMD:R_0402_1005Metric, B.Cu at (74.3, 79.8)
- added TP25: TP4, TestPoint:TestPoint_Pad_D1.0mm, F.Cu at (161.3, 94.1)
- added U4: MSMCP1640T-I/CHY, Package_TO_SOT_SMD:SOT-23-6, B.Cu at (72.0, 79.5)
- C11, C12, C13, C15, C2, C21, C25, C26, C27, C28, C3, C4, C5, C6, D4, J3, L1, Q2, R1, R15, R16, R20, R21, R4, R5, R7, R9, TP23, TP24, TP27, TP28, U2, U3: moved to B.Cu
- L2: value 10uH -> 4.7uH; moved to B.Cu
- Q1: footprint Library:SOT-23-3_L2.9-W1.3-P1.90-LS2.4-BR -> Package_TO_SOT_SMD:SOT-23-3
- Q3, Q4: footprint Library:SOT-23-3_L2.9-W1.3-P1.90-LS2.4-BR -> Package_TO_SOT_SMD:SOT-23-3; moved to B.Cu
- moved J4 73.7 mm to (71.6, 89.8), turned to 180 degrees
- moved BZ1 73.2 mm to (72.7, 81.5), turned to 90 degrees
- moved U2 70.7 mm to (74.1, 74.2), turned to 90 degrees
- moved SW3 68.6 mm to (70.1, 71.4)
- moved SW6 67.1 mm to (76.5, 71.4)
- moved Q4 63.5 mm to (76.5, 79.5), turned to -90 degrees
- moved SW5 62.5 mm to (92.8, 71.5), turned to 180 degrees
- moved R23 61.1 mm to (73.2, 73.6), turned to 180 degrees
- moved R9 60.1 mm to (70.3, 74.8), turned to 90 degrees
- moved Q3 59.1 mm to (76.5, 83.8), turned to -90 degrees
- moved C24 58.6 mm to (71.3, 73.6)
- moved R21 58.3 mm to (74.3, 77.8), turned to 90 degrees
- moved R1 58.0 mm to (82.0, 74.8), turned to 90 degrees
- moved SW4 57.5 mm to (84.3, 71.4)
- moved R20 57.0 mm to (74.3, 83.8), turned to -90 degrees
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Connections:
- net /USB2_DN renamed /USB2_D-
- net /USB2_DP renamed /USB2_D+
- TP25 pad 1: /I2C_SCL -> VBUS_OUT
- U1 pad 1: unconnected-(U1-PB9-Pad1) -> /BUCK_PG
- U1 pad 11: /BUCK_PG -> unconnected-(U1-PA4-Pad11)
- U1 pad 12: unconnected-(U1-PA5-Pad12) -> /BTN_AUX
- U1 pad 14: /BTN_AUX -> /BTN_PAGE
- U1 pad 21: unconnected-(U1-PA10-Pad21) -> /OLED_RESET
- U1 pad 7: /BTN_PAGE -> unconnected-(U1-PA0-Pad7)
- U1 pad 9: /OLED_RESET -> unconnected-(U1-PA2-Pad9)
- U2 pad 8: Net-(U2-IN-) -> VBUS_OUT
Routing:
- net /SBU1_PASS: track 0.00 -> 49.1 mm, vias 0 -> 2
- net /CC2_PASS: track 0.00 -> 42.6 mm, vias 0 -> 4
- net /SBU2_PASS: track 0.00 -> 40.9 mm, vias 0 -> 2
- net /CC1_PASS: track 0.00 -> 39.9 mm, vias 0 -> 2
- net /USB2_D-: track 0.00 -> 37.5 mm, vias 0 -> 2
- net /USB2_D+: track 0.00 -> 37.5 mm, vias 0 -> 2
- net /NRST: track 0.00 -> 36.2 mm, vias 0 -> 2
- net /I2C_SDA: track 0.00 -> 32.2 mm, vias 0 -> 1
- net /I2C_SCL: track 0.00 -> 31.8 mm, vias 0 -> 1
- net +3.3V: track 0.00 -> 15.8 mm, vias 0 -> 8
- net /SWCLK: track 0.00 -> 14.8 mm
- net Net-(U3-SW): track 0.00 -> 13.4 mm
- net /INA_ALERT: track 0.00 -> 11.8 mm, vias 0 -> 1
- net OLED_3V8: track 0.00 -> 11.8 mm
- net /BTN_PAGE: track 0.00 -> 10.7 mm
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- added copper zone on B.Cu, net +3.3V
- added copper zone on B.Cu, net Net-(U3-SW)
- added copper zone on B.Cu, net VBUS_IN
- added copper zone on F.Cu, net VBUS_IN
- added copper zone on B.Cu, net VBUS_OUT
- added copper zone on F.Cu, net VBUS_OUT
- added copper zone on In2.Cu, net VBUS_OUT
- added copper zone on B.Cu, net VBUS_SW
Other:
- board outline added: 33.5 x 24 mm
- copper layers 2 -> 4
- board text added: "if u can see me,ts dont work"

Commit message: Fabrication Push
Parts:
- removed TP17: TP4, TestPoint:TestPoint_Pad_D1.0mm
- removed the TP25 at (161.3, 94.1)
- added G***: LOGO, LOGO, F.Cu at (67.7, 76.4)
- added G***: LOGO, LOGO, F.Cu at (84.5, 91.3)
- added G***: LOGO, LOGO, F.Cu at (94.2, 76.1)
- added G***: LOGO, LOGO, B.Cu at (97.8, 81.4)
- added G***: LOGO, LOGO, B.Cu at (65.6, 81.4)
- added G***: LOGO, LOGO, B.Cu at (68.0, 88.4)
- added TP26: TP5, TestPoint:TestPoint_Pad_2.0x2.0mm, F.Cu at (93.2, 91.6)
- TP18, TP20, TP21, TP22, TP25: moved to B.Cu
- TP19: footprint TestPoint:TestPoint_Pad_D1.0mm -> TestPoint:TestPoint_Pad_2.0x2.0mm; moved to B.Cu
- moved TP19 55.2 mm to (94.0, 91.2), turned to 180 degrees
- moved TP25 44.0 mm to (73.8, 70.8), turned to 180 degrees
- moved TP20 43.5 mm to (85.4, 73.8), turned to 180 degrees
- moved TP22 43.0 mm to (71.9, 84.6)
- moved TP21 40.3 mm to (88.4, 71.2)
- moved TP18 25.7 mm to (94.0, 87.8), turned to 0 degrees
- moved C1 6.58 mm to (90.0, 78.1), turned to 90 degrees
- moved TP28 2.31 mm to (69.0, 74.8)
- moved TP27 1.51 mm to (66.6, 74.8)
- moved C16 1.45 mm to (71.0, 82.5)
- moved C5 1.30 mm to (85.7, 76.7), turned to 90 degrees
- moved R24 1.07 mm to (87.4, 73.6), turned to 180 degrees
- moved L2 0.50 mm to (69.8, 78.5)
- moved C18 0.26 mm to (90.2, 80.0)
Routing:
- net +3.3V: track 15.8 -> 68.9 mm, vias 8 -> 17
- net /USB2_D-: track 37.5 -> 49.2 mm, vias 2 -> 3
- net /USB2_D+: track 37.5 -> 49.0 mm, vias 2 -> 3
- net VBUS_OUT: track 7.21 -> 13.3 mm
- net Net-(D4-A): track 9.20 -> 13.9 mm
- net GND: track 0.00 -> 4.63 mm, vias 0 -> 47
- net VBUS_IN: track 0.00 -> 3.57 mm
- net /CC2_PASS: track 42.6 -> 45.8 mm, vias 4 -> 2
- net Net-(U3-SW): track 13.4 -> 16.2 mm, vias 0 -> 2
- net /I2C_SDA: track 32.2 -> 34.1 mm
- net /I2C_SCL: track 31.8 -> 33.7 mm
- net VBUS_SW: track 3.63 -> 4.98 mm
- net /BTN_RESET: track 7.36 -> 6.53 mm
- net /BUCK_PG: track 6.31 -> 6.90 mm
- net /BUCK_BOOT: track 1.77 -> 1.24 mm
- added copper zone on In2.Cu, net +3.3V
- added copper zone on B.Cu, net GND
- added copper zone on F.Cu, net GND
- added copper zone on In1.Cu, net GND
- added copper zone on In2.Cu, net GND
Other:
- board text added: "BTN#1"
- board text added: "BTN#2"
- board text added: "BTN#3"
- board text added: "GND"
- board text added: "JLCJLCJLCJLC"
- board text added: "JYK"
- board text added: "PWR SWITCH"
- board text added: "REV 1.0"
- board text added: "SHUNT"
- board text added: "SSD1315 DISPLAY"
- board text added: "SWD"
- board text added: "USB_PWR_METER"
- board text added: "if u can see me,ts dont work :("
- board text removed: "if u can see me,ts dont work"
